File: telluino-hb-kicad/telluino.kicad_pcb (KiCad board)
At the start: 2 copper layers, 92 parts, among them J1 6P2C, J3 USB_B, J4 USB_A, Q2 MMBT3904, Q4 ZXTP2012Z, SW1 SW_Push, U1 LE9641PQC, U10 SS1P3L, U2 TISP61089BDR-S, U3 SS1P3L, U4 ATmega328P-A, U5 CH340C, U6 SS1P3L, U7 SS1P3L, U8 TXS0108EPWRG4, U9 CH340C, Y1 16MHz

Commit message: first_routing
Parts:
- removed CCS2: 220pF, Capacitor_SMD:C_0603_1608Metric
- removed CFL3: 0.1uF/100V, Capacitor_SMD:C_0603_1608Metric
- removed CFL4: 10uF/100V, Capacitor_THT:CP_Radial_D8.0mm_P3.50mm
- removed CPF3: 0.1uF/100V, Capacitor_SMD:C_0603_1608Metric_Pad1.08x0.95mm_HandSolder
- removed CPF4: 1uF/100V, Capacitor_THT:CP_Radial_D8.0mm_P3.50mm
- removed CS2: 100nF/25V, Capacitor_SMD:C_0603_1608Metric
- removed CSW2: 10uF/25V, Capacitor_SMD:C_0603_1608Metric
- removed CSWB1: 220uF/25V, Capacitor_THT:CP_Radial_D10.0mm_P5.00mm
- removed CV1: 4.7uF/8.3V, Capacitor_SMD:C_0603_1608Metric
- removed CV2: 1uF/8.3V, Capacitor_SMD:C_0603_1608Metric
- removed CVA1: 0.1uF/16V, Capacitor_SMD:C_0603_1608Metric
- removed CVD1: 0.01uF/16V, Capacitor_SMD:C_0603_1608Metric
- removed CVID1: 0.1uF/18V, Capacitor_SMD:C_0603_1608Metric
- removed DSW2: ES1C-13-F 1A/150V, Diode_SMD:D_SMA
- removed F2: MF-MSMF050-2, my_lib:FUSM4632X85
- removed J3: USB_B, Connector_USB:USB_B_Lumberg_2411_02_Horizontal
- removed J4: USB_A, Connector_USB:USB_A_CNCTech_1001-011-01101_Horizontal
- removed JSM1: 77313-101-30LF, my_lib:AMPHENOL_77313-101-30LF
- removed L2: 47uH 1.5A, Inductor_SMD:L_10.4x10.4_H4.8
- removed Q2: MMBT3904, Package_TO_SOT_SMD:SOT-23
- removed Q4: ZXTP2012Z, teluino:SOT-89-3_4P5X2P6_DIO
- removed RB2: 1K, Resistor_SMD:R_0603_1608Metric
- removed RC2: 75R, Resistor_SMD:R_0603_1608Metric
- removed RCPM1, RCPM2, RS1, RTDC1, RTDC2: 1Meg 1%, Resistor_SMD:R_0603_1608Metric
- removed RCS2: 3.48K, Resistor_SMD:R_0402_1005Metric
- removed RE2: 75R 5%, Resistor_SMD:R_0603_1608Metric
- removed RLM5, RLM6, RLM7, RLM8: 1R0 1/16W, Resistor_SMD:R_0402_1005Metric
- removed RN2: 4*1K, my_lib:SOIC127P780X210-8N
- removed RP2: 10K, Resistor_SMD:R_0603_1608Metric
- removed RPF2: 20R, Resistor_SMD:R_1206_3216Metric
- removed RREF1: 75K 0.5%, Resistor_SMD:R_0603_1608Metric
- removed RT1: 47.5K 1%, Resistor_SMD:R_0603_1608Metric
- removed RTAC1, RTAC2: 10K 1%, Resistor_SMD:R_0603_1608Metric
- removed RTH2: 1K, Resistor_SMD:R_0402_1005Metric
- removed RV1: 2R0 5%, Resistor_SMD:R_0603_1608Metric
- removed RVP1: 0, Resistor_SMD:R_0603_1608Metric
- removed SW1: SW_Push, Button_Switch_SMD:SW_SPST_TL3305A
- removed U10, U6, U7: SS1P3L, my_lib:DO220AAL
- removed U5, U9: CH340C, Package_SO:SOIC-16_3.9x9.9mm_P1.27mm
- removed U8: TXS0108EPWRG4, my_lib:SOP65P640X120-20N
- removed Y1: 16MHz, Crystal:Crystal_HC49-U-3Pin_Vertical
- added C14: 10uF/100V, Capacitor_THT:CP_Radial_D8.0mm_P3.50mm, F.Cu at (121.9, 81.2)
- added C24: 0.1uF, Capacitor_SMD:C_0603_1608Metric, B.Cu at (169.0, 108.0)
- added C31: 0.1 uF/16V, Capacitor_SMD:C_0603_1608Metric, F.Cu at (125.0, 101.8)
- added C35: 0.1 uF/16V, Capacitor_SMD:C_0603_1608Metric, F.Cu at (111.3, 105.1)
- added D8: SS1P3L, my_lib:DO220AAL, F.Cu at (157.0, 103.8)
- added D9: ES1C-13-F 1A/150V, Diode_SMD:D_SMA, F.Cu at (154.8, 92.8)
- added J2: USB_A, Connector_USB:USB_A_CNCTech_1001-011-01101_Horizontal, F.Cu at (190.2, 96.0)
- added JLEFT1: SSQ-115-01-F-S, my_lib:SAMTEC_SSQ-115-01-F-S, B.Cu at (150.1, 111.6)
- added JRIGHT1: SSQ-115-01-F-S, my_lib:SAMTEC_SSQ-115-01-F-S, B.Cu at (150.1, 96.4)
- added L1: 47uH 1.5A, Inductor_SMD:L_10.4x10.4_H4.8, F.Cu at (151.1, 85.0)
- added Q1: MMBT3904, Package_TO_SOT_SMD:SOT-23, F.Cu at (132.3, 83.4)
- added R1: 1Meg 1%, Resistor_SMD:R_0603_1608Metric, F.Cu at (114.2, 111.9)
- added R10: 75K 0.5%, Resistor_SMD:R_0603_1608Metric, F.Cu at (117.1, 95.7)
- added R11: 10K, Resistor_SMD:R_0603_1608Metric, F.Cu at (130.3, 100.1)
- added R12: 75R 5%, Resistor_SMD:R_0603_1608Metric, F.Cu at (128.5, 84.5)
- added R13: 75R, Resistor_SMD:R_0603_1608Metric, F.Cu at (133.6, 87.0)
- added R14: 1K, Resistor_SMD:R_0603_1608Metric, F.Cu at (131.8, 87.0)
- added R15: 1R0 1/16W, Resistor_SMD:R_0402_1005Metric, F.Cu at (147.4, 92.8)
- added R16: 1R0 1/16W, Resistor_SMD:R_0402_1005Metric, F.Cu at (146.1, 92.8)
- added R17: 1R0 1/16W, Resistor_SMD:R_0402_1005Metric, F.Cu at (144.8, 92.8)
- added R18: 1R0 1/16W, Resistor_SMD:R_0402_1005Metric, F.Cu at (143.6, 92.8)
- added R19: 3.48K, Resistor_SMD:R_0402_1005Metric, F.Cu at (127.0, 105.6)
- added R2: 1Meg 1%, Resistor_SMD:R_0603_1608Metric, F.Cu at (112.5, 111.9)
- added R20: 1K, Resistor_SMD:R_0402_1005Metric, F.Cu at (125.7, 105.6)
- added R21: 20R, Resistor_SMD:R_1206_3216Metric, F.Cu at (160.4, 92.1)
- added R22: 2R0 5%, Resistor_SMD:R_0603_1608Metric, F.Cu at (124.2, 94.9)
- added R3: 0, Resistor_SMD:R_0603_1608Metric, F.Cu at (111.3, 103.3)
- added R4: 1Meg 1%, Resistor_SMD:R_0603_1608Metric, F.Cu at (117.6, 110.2)
- added R5: 1Meg 1%, Resistor_SMD:R_0603_1608Metric, F.Cu at (121.2, 110.2)
- added R6: 47.5K 1%, Resistor_SMD:R_0603_1608Metric, F.Cu at (111.3, 106.9)
- added R7: 10K 1%, Resistor_SMD:R_0603_1608Metric, F.Cu at (108.2, 108.9)
- added R8: 10K 1%, Resistor_SMD:R_0603_1608Metric, F.Cu at (108.2, 110.7)
- added R9: 1Meg 1%, Resistor_SMD:R_0603_1608Metric, F.Cu at (118.9, 95.7)
- added locked: ZXTP2012Z, teluino:SOT-89-3_4P5X2P6_DIO, F.Cu at (131.3, 91.6)
- C10: value 4.7 uF/8.3V -> 10uF/25V
- C11: value 0.1 uF/16V -> 100nF/25V
- C12: value 0.1uF -> 220uF/25V; footprint Capacitor_SMD:C_0603_1608Metric -> Capacitor_THT:CP_Radial_D10.0mm_P5.00mm
- C13: value 0.1uF -> 0.1uF/100V
- C15: value 10uF_16V -> 0.1uF/100V; footprint Capacitor_THT:CP_Radial_D5.0mm_P2.50mm -> Capacitor_SMD:C_0603_1608Metric_Pad1.08x0.95mm_HandSolder
- C16: value 100nF -> 1uF/100V; footprint Capacitor_SMD:C_0603_1608Metric -> Capacitor_THT:CP_Radial_D8.0mm_P3.50mm
- C17: value 100nF -> 220pF
- C18: value 1uF -> 0.1uF/18V; moved to B.Cu
- C19: value 1uF -> 4.7uF/8.3V
- C20: value 1uF -> 0.01uF/16V
- C21: value 10uF_16V -> 0.1uF/16V; footprint Capacitor_THT:CP_Radial_D5.0mm_P2.50mm -> Capacitor_SMD:C_0603_1608Metric
- C22: value 100nF -> 1uF/8.3V
- C23: value 10uF_16V -> 0.1uF; footprint Capacitor_THT:CP_Radial_D5.0mm_P2.50mm -> Capacitor_SMD:C_0603_1608Metric; moved to B.Cu
- C25: value 0.1uF -> 100nF
- C26: value 0.1uF -> 10uF_16V; footprint Capacitor_SMD:C_0603_1608Metric -> Capacitor_THT:CP_Radial_D5.0mm_P2.50mm
- C7: value 0.1 uF/16V -> 4.7 uF/8.3V
- D1: value PWR Green -> OP1 Blue
- D2: value RUN Blue -> OP2 Orange
- D3: value OP Orange -> Red Rx
- D4: value Red Rx -> Green Tx
- D5, D7: value Green Tx -> SS1P3L; footprint LED_SMD:LED_0603_1608Metric -> my_lib:DO220AAL
- D6: value Red Rx -> SS1P3L; footprint LED_SMD:LED_0603_1608Metric -> my_lib:DO220AAL
- U3: value SS1P3L -> CH340C; footprint my_lib:DO220AAL -> Package_SO:SOIC-16_3.9x9.9mm_P1.27mm; moved to B.Cu
- U4: value ATmega328P-A -> TXS0108EPWRG4; footprint Package_QFP:TQFP-32_7x7mm_P0.8mm -> my_lib:SOP65P640X120-20N; moved to B.Cu
- moved C22 84.3 mm to (115.1, 107.6)
- moved F1 82.6 mm to (175.6, 84.7)
- moved C16 74.3 mm to (112.7, 81.2), turned to -90 degrees
- moved C20 73.2 mm to (125.0, 100.0), turned to 180 degrees
- moved C19 71.1 mm to (131.8, 104.8)
- moved C17 70.8 mm to (124.2, 106.1), turned to -90 degrees
- moved C18 67.8 mm to (125.0, 103.6)
- moved C12 51.3 mm to (140.0, 86.5), turned to 90 degrees
- moved C15 49.7 mm to (117.0, 87.0)
- moved C13 44.3 mm to (150.3, 92.6), turned to 90 degrees
- moved C21 43.1 mm to (115.3, 95.7), turned to -90 degrees
- moved C1 42.0 mm to (114.0, 90.0)
- moved U2 41.8 mm to (120.9, 90.5)
- moved J1 35.8 mm to (107.3, 92.8)
- moved PTC1 32.6 mm to (105.4, 81.5), turned to 90 degrees
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Connections:
- C1 pad 2: AGND -> GNDA
- C10 pad 1: Net-(U1B-VREF) -> +5V
- C10 pad 2: AGND -> GNDA
- C11 pad 1: AGND -> Net-(C11-Pad1)
- C11 pad 2: VBAT -> SWOUTY
- C12 pad 1: DGND -> +5V
- C12 pad 2: +3.3VA -> GNDA
- C13 pad 1: Net-(U5-~{DTR}) -> VBSENSE
- C13 pad 2: /arduino_controller/RESET* -> GNDA
- C15 pad 1: +5VL -> VBAT
- C15 pad 2: DGND -> GNDA
- C16 pad 1: DGND -> GNDA
- C16 pad 2: +5VL -> VBAT
- C17 pad 1: DGND -> SWISY
- C17 pad 2: Net-(U4-AREF) -> GNDA
- C18 pad 1: DGND -> GNDA
- C18 pad 2: +5V -> +3.3V
- C19 pad 1: DGND -> GNDA
- C19 pad 2: +5V -> +3.3V
- C20 pad 1: DGND -> GNDA
- C20 pad 2: +5V -> +3.3V
- C21 pad 1: +5V -> GNDA
- C21 pad 2: DGND -> +3.3VA
- C22 pad 1: DGND -> GNDA
- C22 pad 2: +5VP -> +3.3VA
- C23 pad 1: +5VP -> Net-(U3-~{DTR})
- C23 pad 2: DGND -> /PC6/RESET
- C25 pad 1: Net-(U9-~{DTR}) -> GNDD
- C25 pad 2: /arduino_controller/RESET* -> +5VP
- C26 pad 1: DGND -> +5VP
- C26 pad 2: +3.3VP -> GNDD
- C5 pad 2: AGND -> GNDA
- C6 pad 1: AGND -> GNDA
- C7 pad 1: AGND -> Net-(U1A-IHL1)
- C7 pad 2: Net-(U1B-DVDD1V2) -> Net-(U1B-VREF)
- C8 pad 1: Net-(U1A-IHL1) -> Net-(U1A-LFC)
- C8 pad 2: Net-(U1B-VREF) -> GNDA
- C9 pad 1: Net-(U1A-LFC) -> Net-(U1B-VREF)
- C9 pad 2: AGND -> GNDA
- D1 pad 1: DGND -> GNDD
- D2 pad 1: DGND -> GNDD
- D3 pad 1: DGND -> USB_RX1
- D4 pad 1: Net-(D4-K) -> USB_TX1
- F1 pad 2: +5VL -> +5VP
- JP1 pad 1: AGND -> GNDA
- JP1 pad 2: DGND -> GNDD
- RN1 pad 1: PB0 -> Net-(D4-A)
- RN1 pad 2: /arduino_controller/RUN -> Net-(D3-A)
- RN1 pad 3: +5V -> Net-(D2-A)
- RN1 pad 4: +5V -> Net-(D1-A)
- RN1 pad 5: Net-(D1-A) -> OP1_LED
- RN1 pad 6: /arduino_controller/RESET* -> OP2_LED
- RN1 pad 7: Net-(D2-A) -> +5V
- RN1 pad 8: Net-(D3-A) -> +5V
- U1 pad 14: 3.3V -> +3.3V
- U1 pad 15: 3.3V -> +3.3V
- U1 pad 23: VDDHPI -> +3.3V
- U1 pad 49: AGND -> GNDD
- U2 pad 6: AGND -> GNDA
- U2 pad 7: AGND -> GNDA
- U4 pad 1: PD2 -> DCLK
- U4 pad 10: PD6 -> +3.3V
- U4 pad 11: PD7 -> GNDD
- U4 pad 12: PB0 -> PCLK_5
- U4 pad 13: /arduino_controller/RUN -> DRA_5
- U4 pad 14: CS_N_5 -> DXA_5
- U4 pad 15: DIN_5 -> FS_5
- U4 pad 17: DCLK_5 -> DIN_5
- U4 pad 18: +5V -> CS_N_5
- U4 pad 19: ADC6 -> +5V
- U4 pad 2: PD4 -> +3.3V
- U4 pad 20: Net-(U4-AREF) -> DCLK_5
- U4 pad 3: DGND -> CS_N
- U4 pad 4: +5V -> DIN
- U4 pad 5: DGND -> DOUT
- U4 pad 6: +5V -> FS
- U4 pad 7: Net-(U4-XTAL1/PB6) -> DXA
- U4 pad 8: Net-(U4-XTAL2/PB7) -> DRA
- U4 pad 9: PD5 -> PCLK
Routing:
- net GNDA: track 0.00 -> 71.5 mm
- net Net-(J1-Pad3): track 0.00 -> 41.8 mm, vias 0 -> 1
- net Net-(J1-Pad4): track 0.00 -> 40.6 mm
- net Net-(U1A-RINGD1): track 0.00 -> 36.7 mm
- net Net-(D9-Pad1): track 0.00 -> 35.7 mm
- net Net-(U2-G): track 0.00 -> 2.45 mm
Other:
- board outline added: 90 x 38 mm

Commit message: placement done
Parts:
- removed C12: 220uF/25V, Capacitor_THT:CP_Radial_D10.0mm_P5.00mm
- added H1: MountingHole, MountingHole:MountingHole_4.3mm_M4, F.Cu at (76.3, 107.0)
- added H2: MountingHole, MountingHole:MountingHole_4.3mm_M4, F.Cu at (76.3, 82.7)
- added H3: MountingHole, MountingHole:MountingHole_4.3mm_M4, F.Cu at (209.3, 107.0)
- added H4: MountingHole, MountingHole:MountingHole_2.2mm_M2, F.Cu at (212.3, 80.0)
- added H5: MountingHole, MountingHole:MountingHole_2.2mm_M2, F.Cu at (162.3, 103.0)
- C18, JLEFT1, JRIGHT1, U4: moved to F.Cu
- moved C16 46.8 mm to (153.8, 103.4), turned to 90 degrees
- moved R21 42.0 mm to (120.5, 105.3), turned to 180 degrees
- moved C26 41.5 mm to (209.9, 85.7)
- moved JLEFT1 40.1 mm to (178.7, 83.5)
- moved C15 38.0 mm to (153.8, 96.5)
- moved D7 37.6 mm to (193.9, 94.7), turned to -90 degrees
- moved RN1 37.3 mm to (199.3, 91.9), turned to 90 degrees
- moved D8 35.1 mm to (190.9, 94.6), turned to -90 degrees
- moved D6 32.8 mm to (200.3, 83.2)
- moved C14 32.0 mm to (144.9, 103.4), turned to 90 degrees
- moved D9 31.7 mm to (124.9, 103.1), turned to -90 degrees
- moved C25 30.6 mm to (205.1, 81.7)
- moved D1 30.4 mm to (201.2, 105.6), turned to 90 degrees
- moved F1 29.0 mm to (204.6, 86.3), turned to 90 degrees
- moved JRIGHT1 28.7 mm to (178.7, 98.7)
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Connections:
- net Net-(U1A-RINGD1) renamed /RING
- net Net-(U1A-TIPD1) renamed /TIP
- J1 pad 3: Net-(J1-Pad3) -> /RING_IN
- J1 pad 4: Net-(J1-Pad4) -> /TIP_IN
- JLEFT1 pad 07: USB_RX1 -> USB_TX1
- JLEFT1 pad 08: USB_TX1 -> USB_RX1
- JLEFT1 pad 11: OP1_LED -> OP2_LED
- JLEFT1 pad 12: OP2_LED -> OP1_LED
- PTC1 pad 1: Net-(J1-Pad4) -> /RING_IN
- PTC1 pad 3: Net-(J1-Pad3) -> /TIP_IN
- R1 pad 1: Net-(J1-Pad3) -> /RING_IN
- R2 pad 1: Net-(J1-Pad4) -> /TIP_IN
- RN1 pad 1: Net-(D4-A) -> Net-(D3-A)
- RN1 pad 2: Net-(D3-A) -> Net-(D4-A)
- U4 pad 1: DCLK -> CS_N
- U4 pad 12: PCLK_5 -> FS_5
- U4 pad 13: DRA_5 -> DXA_5
- U4 pad 14: DXA_5 -> DRA_5
- U4 pad 15: FS_5 -> PCLK_5
- U4 pad 16: DOUT_5 -> DCLK_5
- U4 pad 18: CS_N_5 -> DOUT_5
- U4 pad 20: DCLK_5 -> CS_N_5
- U4 pad 3: CS_N -> DOUT
- U4 pad 5: DOUT -> DCLK
- U4 pad 6: FS -> PCLK
- U4 pad 7: DXA -> DRA
- U4 pad 8: DRA -> DXA
- U4 pad 9: PCLK -> FS
Routing:
- net GNDD: track 0.00 -> 208.1 mm, vias 0 -> 17
- net +5V: track 0.00 -> 170.0 mm, vias 0 -> 5
- net +3.3V: track 0.00 -> 153.9 mm, vias 0 -> 8
- net GNDA: track 71.5 -> 191.8 mm, vias 0 -> 6
- net DCLK_5: track 0.00 -> 83.4 mm, vias 0 -> 2
- net FS_5: track 0.00 -> 70.9 mm, vias 0 -> 2
- net INT_N: track 0.00 -> 69.4 mm, vias 0 -> 4
- net VBAT: track 0.00 -> 65.8 mm, vias 0 -> 2
- net DOUT_5: track 0.00 -> 65.6 mm
- net DXA_5: track 0.00 -> 64.7 mm, vias 0 -> 2
- net DIN_5: track 0.00 -> 62.4 mm
- net CS_N_5: track 0.00 -> 61.3 mm, vias 0 -> 1
- net DRA_5: track 0.00 -> 48.1 mm
- net PCLK_5: track 0.00 -> 46.9 mm, vias 0 -> 2
- net USB_TX1: track 0.00 -> 43.9 mm, vias 0 -> 3
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Other:
- board size 90 x 38 mm -> 143 x 34 mm

Commit message: final board
Parts:
- moved R2 7.82 mm to (94.3, 108.0)
- moved C10 7.82 mm to (112.3, 93.9)
- moved C14 7.82 mm to (149.6, 109.7)
- moved C16 7.82 mm to (158.5, 109.7)
- moved R10 7.82 mm to (111.5, 96.3)
- moved C21 7.82 mm to (109.8, 96.3)
- moved C1 7.82 mm to (95.8, 92.1)
- moved C11 7.82 mm to (145.6, 102.2)
- moved C13 7.82 mm to (144.6, 110.6)
- moved C15 7.82 mm to (158.5, 102.7)
- moved C17 7.82 mm to (119.2, 108.3)
- moved C18 7.82 mm to (123.5, 106.5)
- moved C19 7.82 mm to (120.4, 106.8)
- moved C20 7.82 mm to (120.4, 98.9)
- moved C23 7.82 mm to (183.4, 102.7)
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Routing:
- net Net-(D9-Pad1): track 28.4 -> 29.2 mm
- added copper zone on B.Cu, net GNDA
- added copper zone on F.Cu, net GNDD
Other:
- board text added: "(c) All rights reserved to luis.coelho720813@gmail.com"
- board text added: "2013.06 Telluino V1.0 by Ksoft"

Commit message: order_made
Parts:
- removed H4: MountingHole, MountingHole:MountingHole_2.2mm_M2
- added JP2: A_D_Ground_Bridge, Jumper:SolderJumper-2_P1.3mm_Bridged_RoundedPad1.0x1.5mm, B.Cu at (124.8, 94.1)
- added V1.0: MyLogo, my_lib:MyLogo, F.Cu at (169.0, 113.4)
- locked: footprint teluino:SOT-89-3_4P5X2P6_DIO -> my_lib:SOT-89-3_4P5X2P6_DIO
- moved R10 0.09 mm to (111.5, 96.3)
- moved D5 0.06 mm to (171.7, 101.4)
Routing:
- net VBSENSE: track 38.3 -> 49.6 mm
- net GNDA: track 191.8 -> 200.8 mm
- net GNDD: track 208.1 -> 215.9 mm, vias 17 -> 19
- net +3.3V: track 153.9 -> 157.9 mm
- net Net-(L1-Pad2): track 22.6 -> 26.5 mm
- net +3.3VA: track 29.4 -> 33.2 mm
- net +5V: track 170.0 -> 167.9 mm
- net /TIP_IN: track 22.7 -> 24.7 mm
- net VBAT: track 65.8 -> 64.1 mm
- net /TIP: track 35.9 -> 34.6 mm
- net DOUT_5: track 65.6 -> 64.6 mm
- net /RING_IN: track 42.4 -> 41.7 mm
- net Net-(U1A-RTV1): track 8.35 -> 7.75 mm
- net Net-(D9-Pad1): track 29.2 -> 28.6 mm
- net USB_TX1: track 43.9 -> 43.3 mm
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- added copper zone on F.Cu, net GNDA
- added copper zone on B.Cu, net GNDD
