File: telluino-hb-kicad/telluino.kicad_sch (KiCad schematic)
At the start: 0 parts

Commit message: first_routing
Parts:
- added C1: 0.1 uF/100V, Capacitor_SMD:C_0603_1608Metric, symbol Device:C_Small
- added C10: 10uF/25V, Capacitor_SMD:C_0603_1608Metric, symbol Device:C_Small
- added C11: 100nF/25V, Capacitor_SMD:C_0603_1608Metric, symbol Device:C_Small
- added C12: 220uF/25V, Capacitor_THT:CP_Radial_D10.0mm_P5.00mm, symbol Device:C_Polarized_US
- added C13: 0.1uF/100V, Capacitor_SMD:C_0603_1608Metric, symbol Device:C_Small
- added C14: 10uF/100V, Capacitor_THT:CP_Radial_D8.0mm_P3.50mm, symbol Device:C_Polarized_US
- added C15: 0.1uF/100V, Capacitor_SMD:C_0603_1608Metric_Pad1.08x0.95mm_HandSolder, symbol Device:C_Small
- added C16: 1uF/100V, Capacitor_THT:CP_Radial_D8.0mm_P3.50mm, symbol Device:C_Polarized_US
- added C17: 220pF, Capacitor_SMD:C_0603_1608Metric, symbol Device:C_Small
- added C18: 0.1uF/18V, Capacitor_SMD:C_0603_1608Metric, symbol Device:C_Small
- added C19: 4.7uF/8.3V, Capacitor_SMD:C_0603_1608Metric, symbol Device:C_Small
- added C2, C3, C4, C5, C6: 22 nF/100V, Capacitor_SMD:C_0603_1608Metric, symbol Device:C_Small
- added C20: 0.01uF/16V, Capacitor_SMD:C_0603_1608Metric, symbol Device:C_Small
- added C21: 0.1uF/16V, Capacitor_SMD:C_0603_1608Metric, symbol Device:C_Small
- added C22: 100nF, Capacitor_SMD:C_0603_1608Metric, symbol Device:C_Small
- added C22: 1uF/8.3V, Capacitor_SMD:C_0603_1608Metric, symbol Device:C_Small
- added C23: 10uF_16V, Capacitor_THT:CP_Radial_D5.0mm_P2.50mm, symbol Device:C_Polarized_Small
- added C25, C26: 0.1uF, Capacitor_SMD:C_0603_1608Metric, symbol Device:C_Small
- added C31, C35: 0.1 uF/16V, Capacitor_SMD:C_0603_1608Metric, symbol Device:C_Small
- added C7, C8, C9: 4.7 uF/8.3V, Capacitor_SMD:C_0603_1608Metric, symbol Device:C_Small
- added D3: OP2 Orange, LED_SMD:LED_0603_1608Metric, symbol Device:LED
- added D3: OP1 Blue, LED_SMD:LED_0603_1608Metric, symbol Device:LED
- added D6: Red Rx, LED_SMD:LED_0603_1608Metric, symbol Device:LED
- added D7: Green Tx, LED_SMD:LED_0603_1608Metric, symbol Device:LED
- added D9: ES1C-13-F 1A/150V, Diode_SMD:D_SMA, symbol teluino2:ES1C-13-F
- added F2: MF-MSMF050-2, my_lib:FUSM4632X85, symbol MSMF050:MF-MSMF050-2
- added J1: 6P2C, Connector_RJ:RJ12_Amphenol_54601, symbol my_lib:6P2C
- added J4: USB_A, Connector_USB:USB_A_CNCTech_1001-011-01101_Horizontal, symbol Connector:USB_A
- added JLEFT1, JRIGHT1: SSQ-115-01-F-S, my_lib:SAMTEC_SSQ-115-01-F-S, symbol pin_15_01:SSQ-115-01-F-S
- added JP1: A_D_Ground_Bridge, Jumper:SolderJumper-2_P1.3mm_Bridged_RoundedPad1.0x1.5mm, symbol Jumper:SolderJumper_2_Bridged
- added L1: 47uH 1.5A, Inductor_SMD:L_10.4x10.4_H4.8, symbol Device:L_Ferrite
- added PTC1: MF-SD013, my_lib:ptc-4-mf-sd, symbol my_lib:MF-SD013/250
- added Q1: MMBT3904, Package_TO_SOT_SMD:SOT-23, symbol Transistor_BJT:MMBT3904
- added Q2: ZXTP2012Z, teluino:SOT-89-3_4P5X2P6_DIO, symbol teluino:ZXTP2012Z
- added R1, R2, R4, R5, R9: 1Meg 1%, Resistor_SMD:R_0603_1608Metric, symbol Device:R
- added R10: 75K 0.5%, Resistor_SMD:R_0603_1608Metric, symbol Device:R_Small
- added R11: 10K, Resistor_SMD:R_0603_1608Metric, symbol Device:R
- added R12: 75R 5%, Resistor_SMD:R_0603_1608Metric, symbol Device:R
- added R13: 75R, Resistor_SMD:R_0603_1608Metric, symbol Device:R
- added R14: 1K, Resistor_SMD:R_0603_1608Metric, symbol Device:R
- added R15, R16, R17, R18: 1R0 1/16W, Resistor_SMD:R_0402_1005Metric, symbol Device:R
- added R19: 3.48K, Resistor_SMD:R_0402_1005Metric, symbol Device:R
- added R20: 1K, Resistor_SMD:R_0402_1005Metric, symbol Device:R
- added R21: 20R, Resistor_SMD:R_1206_3216Metric, symbol Device:R
- added R22: 2R0 5%, Resistor_SMD:R_0603_1608Metric, symbol Device:R_Small
- added R3: 0, Resistor_SMD:R_0603_1608Metric, symbol Device:R_Small
- added R6: 47.5K 1%, Resistor_SMD:R_0603_1608Metric, symbol Device:R_Small
- added R7, R8: 10K 1%, Resistor_SMD:R_0603_1608Metric, symbol Device:R_Small
- added RN2: 4*1K, my_lib:SOIC127P780X210-8N, symbol Device:R_Pack04
- added U1: LE9641PQC, my_lib:QFN50P700X700X90-49N, symbol LE9641:LE9641PQC
- added U10, U3, U6, U7: SS1P3L, my_lib:DO220AAL, symbol SS1P3L:SS1P3L
- added U2: TISP61089BDR-S, my_lib:SOIC127P780X210-8N, symbol TISP61089BDR-S:TISP61089BDR-S
- added U4: TXS0108EPWRG4, my_lib:SOP65P640X120-20N, symbol TXS0108:TXS0108EPWRG4
- added U9: CH340C, Package_SO:SOIC-16_3.9x9.9mm_P1.27mm, symbol Interface_USB:CH340C
Connections:
- new net: Q1.2 (E), R12.2
- new net: J1.4, PTC1.1 (R1), R2.1
- new net: R2.2, U1.8 (TDC1)
- new net: C8.1, U1.10 (LFC)
- new net: L1.2, R15.1, R16.1, R17.1, R18.1, R19.1
- new net: C3.2, R7.1
- new net: R7.2, U1.7 (RAC1)
- new net: C31.2, U1.22 (DVDD1V2)
- new net: D7.2 (A), RN2.1 (R1.1)
- new net: R9.1, U1.31 (I/O1/VS1)
- new net: D6.2 (A), RN2.2 (R2.1)
- new net: C7.2, C9.1, U1.4 (VREF)
- new net: C4.1, C5.1, PTC1.2 (R1), U1.45 (RINGD1), U2.1 (K1), U2.8 (K1)
- new net: C1.1, R3.2, U2.2 (G)
- new net: C3.1, C6.2, PTC1.4 (R2), U1.46 (TIPD1), U2.4 (K2), U2.5 (K2)
- new net: C4.2, R8.1
- new net: R8.2, U1.6 (TAC1)
- new net: C25.1, U9.13 (~{DTR})
- new net: Q1.3 (C), R13.2
- new net: C11.1, Q2.1, R13.1, R14.2
- new net: D9.1, L1.1, Q2.2
- new net: C2.2, R5.1
- new net: R5.2, U1.12 (SWCMPY)
- new net: F2.1, J4.1 (VBUS)
- new net: C7.1, U1.5 (IHL1)
- new net: J4.2 (D-), U9.6 (UD-)
- new net: J4.3 (D+), U9.5 (UD+)
- new net: J1.3, PTC1.3 (R2), R1.1
- new net: R1.2, U1.9 (RDC1)
- new net: D3.2 (A), RN2.3 (R3.1)
- new net: R10.1, U1.33 (IREF)
- new net: D3.2 (A), RN2.4 (R4.1)
- new net: C2.1, R4.2, U1.11 (SWVSY)
- new net: R6.1, U1.1 (RSN1)
- new net: R6.2, U1.3 (RTV1)
- new net +3.3V: C18.2, C19.2, C20.2, Q1.1 (B), R11.1, R22.1, U1.14 (VDDSW), U1.15 (DVDD), U1.23 (VDDHPI), U10.P$1 (K), U4.10 (OE), U4.2 (VCCA), U7.P$1 (K)
- new net +3.3VA: C21.2, C22.2, R22.2, U1.2 (AVDD1), U1.35 (AVDD2)
- new net +3.3VP: C26.2, U10.P$2 (A), U9.4 (V3)
- new net +3V3: JRIGHT1.14, U7.P$2 (A)
- new net +5V: C10.1, C12.1, Q2.3, R14.1, R9.2, RN2.7 (R2.2), RN2.8 (R1.2), U3.P$1 (K), U4.19 (VCCB), U6.P$1 (K), U9.16 (VCC)
- new net +5VL: JRIGHT1.04, U6.P$2 (A)
- new net +5VP: C22.2, C23.1, F2.2, U3.P$2 (A)
- new net ADC6: JRIGHT1.05
- new net ADC7: JRIGHT1.06
- new net AREF: JRIGHT1.13
- new net CS_N: U1.29 (*CS), U4.3 (A2)
- new net CS_N_5: JLEFT1.13, U4.18 (B2)
- new net D0/PD0/RX: JLEFT1.02
- new net D1/PD1/TX: JLEFT1.01
- new net DCLK: U1.26 (DCLK), U4.1 (A1)
- new net DCLK_5: JRIGHT1.15, U4.20 (B1)
- new net DIN: U1.27 (DIN), U4.4 (A3)
- new net DIN_5: JLEFT1.14, U4.17 (B3)
- new net DOUT: U1.28 (DOUT), U4.5 (A4)
- new net DOUT_5: JLEFT1.15, U4.16 (B4)
- new net DRA: U1.20 (DRA/ZMOSI), U4.8 (A7)
- new net DRA_5: JRIGHT1.08, U4.13 (B7)
- new net DXA: U1.19 (DXA/ZMISO), U4.7 (A6)
- new net DXA_5: JRIGHT1.09, U4.14 (B6)
- new net FS: U1.18 (FS/ZSYNC), U4.6 (A5)
- new net FS_5: JRIGHT1.10, U4.15 (B5)
- new net GNDA: C1.2, C10.2, C12.2, C13.2, C14.1, C15.2, C16.1, C17.2, C18.1, C19.1, C20.1, C21.1, C22.1, C35.1, C5.2, C6.1, C8.2, C9.2, JP1.1 (A), R10.2, R15.2, R16.2, R17.2, R18.2, R20.2, U2.6 (A), U2.7 (A)
- new net GNDD: C22.1, C23.2, C26.1, C31.1, D3.1 (K), D3.1 (K), J4.4 (GND), J4.5 (Shield), JLEFT1.04, JP1.2 (B), JRIGHT1.02, U1.49 (GND), U4.11 (GND), U9.1 (GND)
- new net INT_N: JLEFT1.05, U1.25 (*INT)
- new net OP1_LED: JLEFT1.11, RN2.5 (R4.2)
- new net OP2_LED: JLEFT1.12, RN2.6 (R3.2)
- new net PC0: JRIGHT1.12
- new net PC1: JRIGHT1.11
- new net PC6/RESET: C25.2, JLEFT1.03
- new net PCLK: U1.21 (PCLK/ZCLK), U4.9 (A8)
- new net PCLK_5: JRIGHT1.07, U4.12 (B8)
- new net PD3: JLEFT1.06
- new net PD6: JLEFT1.09
- new net PD7: JLEFT1.10
- new net RESET: JRIGHT1.03
- new net SWISY: C17.1, R19.2, R20.1, U1.13 (SWISY)
- new net SWOUTY: C11.2, R11.2, R12.1, U1.16 (SWOUTY)
- new net USB_RX1: D6.1 (K), JLEFT1.07, U9.3 (RXD)
- new net USB_TX1: D7.1 (K), JLEFT1.08, U9.2 (TXD)
- new net VBAT: C15.1, C16.2, C35.2, R21.2, R3.1, U1.48 (VBAT1)
- new net VBSENSE: C13.1, C14.2, D9.2, R21.1, R4.1
- new net VDDHPI: U1.24 (*ZSI)
Other:
- removed sheet arduino_controller
- removed sheet buck_boost_suplly
- removed sheet connectors
- removed sheet slic
- note added: "Buck Boost SUpply"
- note added: "DNP"
- note added: "Locate C20 near DVDD and C21 near AVDD pins."
- note added: "Place Near mSCLIC DEVICE"
- company: (none) -> Ksoft
- title: (none) -> Telluino Hardware-Bottom

Commit message: placement done
Parts:
- removed C12: 220uF/25V, Capacitor_THT:CP_Radial_D10.0mm_P5.00mm, symbol Device:C_Polarized_US
- added H1, H2, H3: MountingHole, MountingHole:MountingHole_4.3mm_M4, symbol Mechanical:MountingHole
- added H4, H5: MountingHole, MountingHole:MountingHole_2.2mm_M2, symbol Mechanical:MountingHole
- renumbered C25 to C23, C26 to C24, C22 to C25, C23 to C26, D3 to D1, D3 to D2, D6 to D3, D7 to D4, U6 to D5, U3 to D6, U7 to D7, U10 to D8, F2 to F1, J4 to J2, RN2 to RN1, U9 to U3
Connections:
- net CS_N: now also U4.1 (A1); no longer U4.3 (A2)
- net CS_N_5: now also U4.20 (B1); no longer U4.18 (B2)
- net DCLK: now also U4.5 (A4); no longer U4.1 (A1)
- net DCLK_5: now also U4.16 (B4); no longer U4.20 (B1)
- net DOUT: now also U4.3 (A2); no longer U4.5 (A4)
- net DOUT_5: now also U4.18 (B2); no longer U4.16 (B4)
- net DRA: now also U4.7 (A6); no longer U4.8 (A7)
- net DRA_5: now also U4.14 (B6); no longer U4.13 (B7)
- net DXA: now also U4.8 (A7); no longer U4.7 (A6)
- net DXA_5: now also U4.13 (B7); no longer U4.14 (B6)
- net FS: now also U4.9 (A8); no longer U4.6 (A5)
- net FS_5: now also U4.12 (B8); no longer U4.15 (B5)
- net OP1_LED: now also JLEFT1.12; no longer JLEFT1.11
- net OP2_LED: now also JLEFT1.11; no longer JLEFT1.12
- net PCLK: now also U4.6 (A5); no longer U4.9 (A8)
- net PCLK_5: now also U4.15 (B5); no longer U4.12 (B8)
- net USB_RX1: now also JLEFT1.08; no longer JLEFT1.07
- net USB_TX1: now also JLEFT1.07; no longer JLEFT1.08
- net TIP_IN: now reaches J1.4, R2.1
- net TIP_IN: now also PTC1.3 (R2); no longer PTC1.1 (R1)
- net at D4.2 (A): now also RN1.2 (R2.1); no longer RN1.1 (R1.1)
- net at D3.2 (A): now also RN1.1 (R1.1); no longer RN1.2 (R2.1)
- net RING: now reaches C4.1, C5.1, PTC1.2 (R1), U1.45 (RINGD1), U2.1 (K1), U2.8 (K1)
- net TIP: now reaches C3.1, C6.2, PTC1.4 (R2), U1.46 (TIPD1), U2.4 (K2), U2.5 (K2)
- net RING_IN: now reaches J1.3, R1.1
- net RING_IN: now also PTC1.1 (R1); no longer PTC1.3 (R2)
Other:
- moved on the sheet: D4

Commit message: order_made
Parts:
- removed H4: MountingHole, MountingHole:MountingHole_2.2mm_M2, symbol Mechanical:MountingHole
- added JP2: A_D_Ground_Bridge, Jumper:SolderJumper-2_P1.3mm_Bridged_RoundedPad1.0x1.5mm, symbol Jumper:SolderJumper_2_Bridged
- C16: now not fitted
- Q2: footprint teluino:SOT-89-3_4P5X2P6_DIO -> my_lib:SOT-89-3_4P5X2P6_DIO
Connections:
- net +3.3V: now also D7.1 (K), D8.1 (K); no longer D7.P$1 (K), D8.P$1 (K)
- net +3.3VP: now also D8.2 (A); no longer D8.P$2 (A)
- net +3V3: now also D7.2 (A); no longer D7.P$2 (A)
- net +5V: now also D5.1 (K), D6.1 (K); no longer D5.P$1 (K), D6.P$1 (K)
- net +5VL: now also D5.2 (A); no longer D5.P$2 (A)
- net +5VP: now also D6.2 (A); no longer D6.P$2 (A)
- net GNDA: now also JP2.1 (A)
- net GNDD: now also JP2.2 (B)
Changed lines of the file:
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@@
   (junction (at 265.43 58.42) (diameter 0) (color 0 0 0 0)
   )
+  (junction (at 138.43 245.11) (diameter 0) (color 0 0 0 0)
+  )
   (junction (at 123.19 152.4) (diameter 0) (color 0 0 0 0)
   )
@@
   (junction (at 264.16 228.6) (diameter 0) (color 0 0 0 0)
   )
+  (junction (at 128.27 245.11) (diameter 0) (color 0 0 0 0)
+  )
   (junction (at 143.51 152.4) (diameter 0) (color 0 0 0 0)
   )
@@
     (stroke (width 0) (type default))
   )
+  (wire (pts (xy 129.54 237.49) (xy 128.27 237.49))
+    (stroke (width 0) (type default))
+  )
   (wire (pts (xy 369.57 39.37) (xy 355.6 39.37))
     (stroke (width 0) (type default))
@@
     (stroke (width 0) (type default))
   )
+  (wire (pts (xy 137.16 237.49) (xy 138.43 237.49))
+    (stroke (width 0) (type default))
+  )
   (wire (pts (xy 68.58 157.48) (xy 68.58 161.29))
     (stroke (width 0) (type default))
@@
     (stroke (width 0) (type default))
   )
+  (wire (pts (xy 201.93 262.89) (xy 204.47 262.89))
+    (stroke (width 0) (type default))
+  )
   (wire (pts (xy 135.89 46.99) (xy 143.51 46.99))
     (stroke (width 0) (type default))
@@
     (stroke (width 0) (type default))
   )
+  (wire (pts (xy 138.43 237.49) (xy 138.43 245.11))
+    (stroke (width 0) (type default))
+  )
   (wire (pts (xy 87.63 255.27) (xy 87.63 259.08))
     (stroke (width 0) (type default))
@@
     (stroke (width 0) (type default))
   )
-  (wire (pts (xy 201.93 262.89) (xy 204.47 262.89))
-    (stroke (width 0) (type default))
-  )
   (wire (pts (xy 41.91 134.62) (xy 54.61 134.62))
     (stroke (width 0) (type default))
@@
     (stroke (width 0) (type default))
   )
+  (wire (pts (xy 128.27 237.49) (xy 128.27 245.11))
+    (stroke (width 0) (type default))
+  )
   (wire (pts (xy 257.81 124.46) (xy 257.81 125.73))
     (stroke (width 0) (type default))
@@
     )
   )
-  (symbol (lib_id "Mechanical:MountingHole") (at 39.37 205.74 0) (unit 1)
-    (in_bom yes) (on_board yes) (dnp no) (fields_autoplaced)
-    (property "Reference" "H4" (at 41.91 205.105 0)
-      (effects (font (size 1.27 1.27)) (justify left))
-    )
-    (property "Value" "MountingHole" (at 41.91 207.645 0)
-      (effects (font (size 1.27 1.27)) (justify left))
-    )
-    (property "Footprint" "MountingHole:MountingHole_2.2mm_M2" (at 39.37 205.74 0)
-      (effects (font (size 1.27 1.27)) hide)
-    )
-    (property "Datasheet" "~" (at 39.37 205.74 0)
-      (effects (font (size 1.27 1.27)) hide)
-    )
-    (instances
-      (project "telluino"
-        (path "/3bd12265-4173-4d6b-91eb-5b474bc7bb16"
-          (reference "H4") (unit 1)
-        )
-      )
-    )
-  )
   (symbol (lib_id "Device:C_Small") (at 226.06 129.54 180) (unit 1)
     (in_bom yes) (on_board yes) (dnp no)
@@
       (effects (font (size 1.524 1.524)) (justify left))
     )
-    (property "Footprint" "teluino:SOT-89-3_4P5X2P6_DIO" (at 71.12 146.05 0)
+    (property "Footprint" "my_lib:SOT-89-3_4P5X2P6_DIO" (at 71.12 146.05 0)
       (effects (font (size 1.27 1.27) italic) hide)
     )
@@
       (effects (font (size 1.27 1.27)) hide)
     )
-    (pin "P$1")
-    (pin "P$2")
+    (pin "1")
+    (pin "2")
     (instances
       (project "telluino"
@@
       (effects (font (size 1.27 1.27)) hide)
     )
-    (pin "P$1")
-    (pin "P$2")
+    (pin "1")
+    (pin "2")
     (instances
       (project "telluino"
@@
     )
   )
+  (symbol (lib_id "Jumper:SolderJumper_2_Bridged") (at 133.35 237.49 0) (unit 1)
+    (in_bom yes) (on_board yes) (dnp no) (fields_autoplaced)
+    (property "Reference" "JP2" (at 133.35 232.41 0)
+      (effects (font (size 1.27 1.27)))
+    )
+    (property "Value" "A_D_Ground_Bridge" (at 133.35 234.95 0)
+      (effects (font (size 1.27 1.27)))
+    )
+    (property "Footprint" "Jumper:SolderJumper-2_P1.3mm_Bridged_RoundedPad1.0x1.5mm" (at 133.35 237.49 0)
+      (effects (font (size 1.27 1.27)) hide)
+    )
+    (property "Datasheet" "~" (at 133.35 237.49 0)
+      (effects (font (size 1.27 1.27)) hide)
+    )
+    (pin "1")
+    (pin "2")
+    (instances
+      (project "telluino"
+        (path "/3bd12265-4173-4d6b-91eb-5b474bc7bb16"
+          (reference "JP2") (unit 1)
+        )
+      )
+    )
+  )
   (symbol (lib_id "Device:LED") (at 185.42 205.74 90) (unit 1)
     (in_bom yes) (on_board yes) (dnp no)
@@
   )
   (symbol (lib_id "Device:C_Polarized_US") (at 154.94 160.02 180) (unit 1)
-    (in_bom yes) (on_board yes) (dnp no)
+    (in_bom yes) (on_board yes) (dnp yes)
     (property "Reference" "C16" (at 161.29 156.21 0)
       (effects (font (size 1.27 1.27)) (justify left))
@@
       (effects (font (size 1.27 1.27)) hide)
     )
-    (pin "P$1")
-    (pin "P$2")
+    (pin "1")
+    (pin "2")
     (instances
       (project "telluino"
@@
       (effects (font (size 1.27 1.27)) hide)
     )
-    (pin "P$1")
-    (pin "P$2")
+    (pin "1")
+    (pin "2")
     (instances
       (project "telluino"

Commit message: small updates
Parts:
- C1: value 0.1 uF/100V -> 0.1uF/100V
- C11: value 100nF/25V -> 0.1uF/100V
- C15: footprint Capacitor_SMD:C_0603_1608Metric_Pad1.08x0.95mm_HandSolder -> Capacitor_SMD:C_0603_1608Metric
- C18: value 0.1uF/18V -> 0.1uF/100V
- C21: value 0.1uF/16V -> 0.1uF/100V
- C22: value 1uF/8.3V -> 1uF/6.3V
- C23, C24: value 0.1uF -> 0.1uF/100V
- C25: value 100nF -> 0.1uF/100V
- C26: value 10uF_16V -> 10uF/25V
- C31, C35: value 0.1 uF/16V -> 0.1uF/100V
- C7, C8, C9: value 4.7 uF/8.3V -> 4.7uF/8.3V
- R10, R22, R3, R6, R7, R8: symbol Device:R_Small -> Device:R
- R11: value 10K -> 10K 1%
- R13: value 75R -> 75R 5%
Connections:
- net +3.3V: no longer R22.1
- net +3.3VA: no longer R22.2
- net VBAT: no longer R3.1
- net at C1.1, U2.2 (G): no longer R3.2
- net at R8.1: no longer C4.2
- net at R8.2: no longer U1.6 (TAC1)
Other:
- moved on the sheet: C35
