File: telluino-hb-kicad/telluino.kicad_sch (KiCad schematic)
At the start: 77 parts, among them J1 6P2C, J2 USB_A, Q1 MMBT3904, Q2 ZXTP2012Z, U1 LE9641PQC, U2 TISP61089BDR-S, U3 CH340C, U4 TXS0108EPWRG4, U5 AMS1117-3.3

Commit message: update_for_next_Version
Connections:
- net +5V: no longer C24.1
- net GNDD: now also C24.1
Changed lines of the file:
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@@
     (stroke (width 0) (type default))
   )
-  (wire (pts (xy 234.95 227.33) (xy 243.84 227.33))
-    (stroke (width 0) (type default))
-  )
   (wire (pts (xy 344.17 115.57) (xy 344.17 165.1))
     (stroke (width 0) (type default))
@@
     (stroke (width 0) (type default))
   )
-  (wire (pts (xy 243.84 227.33) (xy 243.84 215.9))
-    (stroke (width 0) (type default))
-  )
   (wire (pts (xy 148.59 54.61) (xy 151.13 54.61))
     (stroke (width 0) (type default))
@@
     )
   )
+  (symbol (lib_id "power:GNDD") (at 234.95 227.33 0) (unit 1)
+    (in_bom yes) (on_board yes) (dnp no) (fields_autoplaced)
+    (property "Reference" "#PWR018" (at 234.95 233.68 0)
+      (effects (font (size 1.27 1.27)) hide)
+    )
+    (property "Value" "GNDD" (at 234.95 232.41 0)
+      (effects (font (size 1.27 1.27)))
+    )
+    (property "Footprint" "" (at 234.95 227.33 0)
+      (effects (font (size 1.27 1.27)) hide)
+    )
+    (property "Datasheet" "" (at 234.95 227.33 0)
+      (effects (font (size 1.27 1.27)) hide)
+    )
+    (pin "1")
+    (instances
+      (project "telluino"
+        (path "/3bd12265-4173-4d6b-91eb-5b474bc7bb16"
+          (reference "#PWR018") (unit 1)
+        )
+      )
+    )
+  )
   (symbol (lib_id "power:+5V") (at 349.25 107.95 0) (unit 1)
     (in_bom yes) (on_board yes) (dnp no) (fields_autoplaced)
@@
         )
       )
-    )
-  )
-  (symbol (lib_id "power:+5V") (at 243.84 215.9 0) (unit 1)
-    (in_bom yes) (on_board yes) (dnp no) (fields_autoplaced)
-    (property "Reference" "#PWR020" (at 243.84 219.71 0)
-      (effects (font (size 1.27 1.27)) hide)
-    )
-    (property "Value" "+5V" (at 243.84 212.09 0)
-      (effects (font (size 1.27 1.27)))
-    )
-    (property "Footprint" "" (at 243.84 215.9 0)
-      (effects (font (size 1.27 1.27)) hide)
-    )
-    (property "Datasheet" "" (at 243.84 215.9 0)
-      (effects (font (size 1.27 1.27)) hide)
-    )
-    (pin "1")
-    (instances
-      (project "telluino"
-        (path "/3bd12265-4173-4d6b-91eb-5b474bc7bb16"
-          (reference "#PWR020") (unit 1)
-        )
-      )
